File: Power Supply.kicad_sch (KiCad schematic)
At the start: 31 parts, among them J1 Conn_01x04_Socket, P1 Conn_WallPlug, SW1 SW_SPST, T1 36VCT, T2 9V, U1 L7915, U2 L7805, U3 L7815

Commit message: uodates
Parts:
- added J2: Conn_01x04_Socket, Connector_PinHeader_2.54mm:PinHeader_1x04_P2.54mm_Vertical, symbol Connector:Conn_01x04_Socket
- C1, C2, C3, C4, C5, C6: footprint (none) -> Capacitor_THT:CP_Radial_D18.0mm_P7.50mm
- D15: footprint (none) -> LED_THT:LED_D5.0mm
- J1: footprint (none) -> Connector_PinHeader_2.54mm:PinHeader_1x04_P2.54mm_Vertical
- R1: footprint (none) -> Resistor_THT:R_Axial_DIN0614_L14.3mm_D5.7mm_P15.24mm_Horizontal
- U1: footprint (none) -> Library:L7915CV TO255P1040X460X1935-3
- U2: footprint (none) -> Library:L7805 TO255P1020X450X2000-3
- U3: footprint (none) -> Library:L7815CV TO254P450X1020X1935-3P
Connections:
- net at C5.1, D11.1 (K), D6.1 (K)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: no longer C6.1, D11.2 (A), D14.1 (K), J1.4 (Pin_4), U2.3 (OUT)
- net at C4.2, D10.1 (K), D13.2 (A)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: no longer C3.2, D1.2 (A), D10.2 (A), D4.2 (A), U1.2 (VI)
- net at C1.1, D12.1 (K), D9.2 (A)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: no longer C2.1, D2.1 (K), D3.1 (K), D9.1 (K), U3.1 (IN)
- net T1-A: no longer names the net of D1.1 (K), D2.2 (A)
- net T1-A: now also J2.1 (Pin_1); no longer T1.5 (SB)
- net T1-B: no longer names the net of D3.2 (A), D4.1 (K)
- net T1-B: now also J2.2 (Pin_2); no longer T1.3 (SA)
- net T2-A: no longer names the net of D5.1 (K), D6.2 (A)
- net T2-A: now also J2.3 (Pin_3); no longer T2.4 (SB)
- net T2-B: no longer names the net of D7.2 (A), D8.1 (K)
- net T2-B: now also J2.4 (Pin_4); no longer T2.3 (SA)
- new net: C3.2, D1.2 (A), D10.2 (A), D4.2 (A), U1.2 (VI)
- new net: C6.1, D11.2 (A), D14.1 (K), J1.4 (Pin_4), U2.3 (OUT)
- new net: C2.1, D2.1 (K), D3.1 (K), D9.1 (K), U3.1 (IN)
