File: Power Supply.kicad_pcb (KiCad board)
At the start: 2 copper layers, 183 x 42.5 mm, 30 parts, among them J1 Conn_01x04_Socket, J2 Conn_01x04_Socket, U1 L7915, U2 L7805, U3 L7815

Commit message: VCA
Parts:
- removed REF** (x3): Heatsink_Fischer_SK104-STCB_35x13mm__2xDrill3.5mm_ScrewM3, Heatsink:Heatsink_Fischer_SK104-STCB_35x13mm__2xDrill3.5mm_ScrewM3
- added Sink1: Heatsink_Fischer_SK104-STCB_35x13mm__2xDrill1.5mm_ScrewM3, Heatsink:Heatsink_Fischer_SK104-STCB_35x13mm__2xDrill1.5mm_ScrewM3, F.Cu at (136.8, 23.0)
- added Sink2: Heatsink_Fischer_SK104-STCB_35x13mm__2xDrill1.5mm_ScrewM3, Heatsink:Heatsink_Fischer_SK104-STCB_35x13mm__2xDrill1.5mm_ScrewM3, F.Cu at (136.8, 43.0)
- added Sink3: Heatsink_Fischer_SK104-STCB_35x13mm__2xDrill1.5mm_ScrewM3, Heatsink:Heatsink_Fischer_SK104-STCB_35x13mm__2xDrill1.5mm_ScrewM3, F.Cu at (165.0, 34.5)
- moved U2 0.24 mm to (168.9, 34.5)
Routing:
- net GND: track 306.6 -> 97.5 mm, vias 0 -> 6
- net Net-(D10-K): track 165.8 -> 196.0 mm, vias 0 -> 3
- net Net-(D11-K): track 140.1 -> 159.2 mm
- net Net-(D11-A): track 193.5 -> 185.4 mm, vias 0 -> 4
- net Net-(D2-K): track 126.7 -> 120.1 mm
- net Net-(D1-K): track 10.0 -> 15.5 mm
- net Net-(D1-A): track 127.8 -> 124.1 mm, vias 2 -> 0
- net Net-(D12-K): track 136.4 -> 140.1 mm, vias 0 -> 1
- net Net-(D5-K): track 30.5 -> 28.9 mm
- net Net-(D7-A): track 42.5 -> 41.8 mm
- net Net-(D15-K): track 11.8 -> 12.5 mm
- added copper zone on B.Cu, net GND
- added copper zone on F.Cu, net GND
