File: VCA/schematics/mainboard/mainboard.kicad_pcb (KiCad board)
At the start: 2 copper layers, 57.9 x 82.5 mm, 46 parts, among them Q1 BC548, Q2 BC548, Q3 BC548, Q4 BC548, U1 TL072, U2 TL072

Commit message: stuff
Parts:
- added J1: IN 1, Eurorack:AudioJack_3.5mm, F.Cu at (54.5, 65.8)
- added J2: CV 1, Eurorack:AudioJack_3.5mm, F.Cu at (48.9, 122.6)
- added J3: OUT 1, Eurorack:AudioJack_3.5mm, F.Cu at (60.0, 122.6)
- added J4: IN 1, Eurorack:AudioJack_3.5mm, F.Cu at (71.0, 122.6)
- added J5: CV 1, Eurorack:AudioJack_3.5mm, F.Cu at (82.0, 122.6)
- added J6: OUT 1, Eurorack:AudioJack_3.5mm, F.Cu at (93.1, 122.6)
- C1, C2, C3, C4: footprint Capacitor_THT:CP_Radial_D12.5mm_P5.00mm -> Capacitor_THT:CP_Radial_D5.0mm_P2.00mm
- RV2, RV4: footprint Potentiometer_THT:Potentiometer_Bourns_3296W_Vertical -> Eurorack:Potentiometer_RV09
- moved RV4 15.8 mm to (84.2, 110.4)
