File: VCA/schematics/mainboard/mainboard.kicad_sch (KiCad schematic)
At the start: 24 parts, among them J1 AudioJack3, J2 AudioJack3, J3 AudioJack3, Q1 BC548, Q2 BC548, U1 TL072

Commit message: stuff
Parts:
- added C1, C2, C3, C4: 0.1uF, Capacitor_THT:CP_Radial_D12.5mm_P5.00mm, symbol Device:C
- added J4: IN 1, symbol Connector_Audio:AudioJack3
- added J5: CV 1, symbol Connector_Audio:AudioJack3
- added J6: OUT 1, symbol Connector_Audio:AudioJack3
- added Q3, Q4: BC548, Package_TO_SOT_THT:TO-92_Inline, symbol Transistor_BJT:BC548
- added R17, R22, R25: 20k, Resistor_THT:R_Axial_DIN0207_L6.3mm_D2.5mm_P2.54mm_Vertical, symbol Device:R
- added R18, R20, R21, R30, R31: 100k, Resistor_THT:R_Axial_DIN0207_L6.3mm_D2.5mm_P2.54mm_Vertical, symbol Device:R
- added R19: 100, Resistor_THT:R_Axial_DIN0207_L6.3mm_D2.5mm_P2.54mm_Vertical, symbol Device:R
- added R23: 82k, Resistor_THT:R_Axial_DIN0207_L6.3mm_D2.5mm_P2.54mm_Vertical, symbol Device:R
- added R24, R28, R29: 10k, Resistor_THT:R_Axial_DIN0207_L6.3mm_D2.5mm_P2.54mm_Vertical, symbol Device:R
- added R26, R27: R, Resistor_THT:R_Axial_DIN0207_L6.3mm_D2.5mm_P2.54mm_Vertical, symbol Device:R
- added R32: 1k, Resistor_THT:R_Axial_DIN0207_L6.3mm_D2.5mm_P2.54mm_Vertical, symbol Device:R
- added RV3: 100k, Resistor_THT:R_Axial_DIN0207_L6.3mm_D2.5mm_P2.54mm_Vertical, symbol Device:R_Potentiometer
- added RV4: R_Potentiometer, Potentiometer_THT:Potentiometer_Bourns_3296W_Vertical, symbol Device:R_Potentiometer
- added U2: TL072, Package_DIP:DIP-8_W7.62mm, symbol Amplifier_Operational:TL072
- J1: value AudioJack3 -> IN 1
- J2: value AudioJack3 -> CV 1
- J3: value AudioJack3 -> OUT 1
- R1, R8, R9: value R -> 20k; footprint (none) -> Resistor_THT:R_Axial_DIN0207_L6.3mm_D2.5mm_P2.54mm_Vertical
- R10, R11: footprint (none) -> Resistor_THT:R_Axial_DIN0207_L6.3mm_D2.5mm_P2.54mm_Vertical
- R12, R13, R5: value R -> 10k; footprint (none) -> Resistor_THT:R_Axial_DIN0207_L6.3mm_D2.5mm_P2.54mm_Vertical
- R14, R15, R2, R3, R6: value R -> 100k; footprint (none) -> Resistor_THT:R_Axial_DIN0207_L6.3mm_D2.5mm_P2.54mm_Vertical
- R16: value R -> 1k; footprint (none) -> Resistor_THT:R_Axial_DIN0207_L6.3mm_D2.5mm_P2.54mm_Vertical
- R4: value R -> 82k; footprint (none) -> Resistor_THT:R_Axial_DIN0207_L6.3mm_D2.5mm_P2.54mm_Vertical
- R7: value R -> 100; footprint (none) -> Resistor_THT:R_Axial_DIN0207_L6.3mm_D2.5mm_P2.54mm_Vertical
- RV1: value R_Potentiometer -> 100k; footprint (none) -> Resistor_THT:R_Axial_DIN0207_L6.3mm_D2.5mm_P2.54mm_Vertical
- RV2: footprint (none) -> Potentiometer_THT:Potentiometer_Bourns_3296W_Vertical
- U1: footprint (none) -> Package_DIP:DIP-8_W7.62mm
Connections:
- net GND: now also C1.2, C2.1, C3.2, C4.1, J4.S, J5.S, J6.S, R19.2, R26.2, R30.2, RV3.3, U2.3 (+)
- net VCC: now also U1.8 (V+), C1.1, C3.1, R17.1, R22.1, R25.1, R28.1, R29.1, RV4.1, U2.8 (V+)
- net VEE: now also U1.4 (V-), C2.2, C4.2, RV4.3, U2.4 (V-)
- net at J2.T, R3.2: now also J5.R
- net at J1.T, R6.1: now also J4.R
- new net: Q3.3 (E), Q4.3 (E), R24.1
- new net: R23.2, R24.2, U2.1
- new net: R17.2, RV3.1
- new net: Q4.1 (C), R25.2
- new net: Q4.2 (B), R26.1, R27.1
- new net: R28.2, R31.1, U2.5 (+)
- new net: R31.2, R32.1, U2.7
- new net: J6.T, R32.2
- new net: R29.2, R30.1, U2.6 (-)
- new net: Q3.1 (C), R22.2
- new net: J5.T, R21.2
- new net: J4.T, R18.1
- new net: R20.2, R21.1, R23.1, U2.2 (-)
- new net: Q3.2 (B), R18.2, R19.1
- new net: R27.2, RV4.2
- new net: R20.1, RV3.2
Other:
- moved on the sheet: J1, J2, J3, Q1, Q2, R1, R10, R11, R12, R13, R14, R15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

Commit message: stuff
Parts:
- added J7, J8: Conn_01x05_Socket, symbol Connector:Conn_01x05_Socket
- C1, C2, C3, C4: footprint Capacitor_THT:CP_Radial_D12.5mm_P5.00mm -> Capacitor_THT:CP_Radial_D5.0mm_P2.00mm
- J1, J2, J3, J4, J5, J6: footprint (none) -> Eurorack:AudioJack_3.5mm
- RV2, RV4: footprint Potentiometer_THT:Potentiometer_Bourns_3296W_Vertical -> Eurorack:Potentiometer_RV09
Changed lines of the file:
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@@
 			)
 		)
-		(property "Footprint" "Potentiometer_THT:Potentiometer_Bourns_3296W_Vertical"
+		(property "Footprint" "Eurorack:Potentiometer_RV09"
 			(at 146.05 50.8 0)
 			(effects
@@
 			)
 		)
-		(property "Footprint" "Capacitor_THT:CP_Radial_D12.5mm_P5.00mm"
+		(property "Footprint" "Capacitor_THT:CP_Radial_D5.0mm_P2.00mm"
 			(at 110.1852 184.15 0)
 			(effects
@@
 			)
 		)
-		(property "Footprint" "Capacitor_THT:CP_Radial_D12.5mm_P5.00mm"
+		(property "Footprint" "Capacitor_THT:CP_Radial_D5.0mm_P2.00mm"
 			(at 110.1852 191.77 0)
 			(effects
@@
 			)
 		)
-		(property "Footprint" ""
+		(property "Footprint" "Eurorack:AudioJack_3.5mm"
 			(at 66.04 78.74 0)
 			(effects
@@
 			)
 		)
-		(property "Footprint" ""
+		(property "Footprint" "Eurorack:AudioJack_3.5mm"
 			(at 62.23 153.67 0)
 			(effects
@@
 			)
 		)
-		(property "Footprint" ""
+		(property "Footprint" "Eurorack:AudioJack_3.5mm"
 			(at 195.58 31.75 0)
 			(effects
@@
 			)
 		)
-		(property "Footprint" ""
+		(property "Footprint" "Eurorack:AudioJack_3.5mm"
 			(at 62.23 118.11 0)
 			(effects
@@
 			)
 		)
-		(property "Footprint" ""
+		(property "Footprint" "Eurorack:AudioJack_3.5mm"
 			(at 66.04 43.18 0)
 			(effects
@@
 	)
 	(symbol
+		(lib_id "Connector:Conn_01x05_Socket")
+		(at 29.21 90.17 0)
+		(unit 1)
+		(exclude_from_sim no)
+		(in_bom yes)
+		(on_board yes)
+		(dnp no)
+		(fields_autoplaced yes)
+		(property "Reference" "J8"
+			(at 30.48 88.8999 0)
+			(effects
+				(font
+					(size 1.27 1.27)
+				)
+				(justify left)
+			)
+		)
+		(property "Value" "Conn_01x05_Socket"
+			(at 30.48 91.4399 0)
+			(effects
+				(font
+					(size 1.27 1.27)
+				)
+				(justify left)
+				(hide yes)
+			)
+		)
+		(property "Footprint" ""
+			(at 29.21 90.17 0)
+			(effects
+				(font
+					(size 1.27 1.27)
+				)
+				(hide yes)
+			)
+		)
+		(property "Datasheet" "~"
+			(at 29.21 90.17 0)
+			(effects
+				(font
+					(size 1.27 1.27)
+				)
+				(hide yes)
+			)
+		)
+		(property "Description" "Generic connector, single row, 01x05, script generated"
+			(at 29.21 90.17 0)
+			(effects
+				(font
+					(size 1.27 1.27)
+				)
+				(hide yes)
+			)
+		)
+		(pin "5"
+		)
+		(pin "3"
+		)
+		(pin "1"
+		)
+		(pin "2"
+		)
+		(pin "4"
+		)
+		(instances
+			(project ""
+				(path "/d7035e05-04e9-4d00-b42e-d5291b634456"
+					(reference "J8")
+					(unit 1)
+				)
+			)
+		)
+	)
+	(symbol
 		(lib_id "Amplifier_Operational:TL072")
 		(at 128.27 184.15 0)
@@
 			)
 		)
-		(property "Footprint" "Potentiometer_THT:Potentiometer_Bourns_3296W_Vertical"
+		(property "Footprint" "Eurorack:Potentiometer_RV09"
 			(at 142.24 125.73 0)
 			(effects
@@
 	)
 	(symbol
+		(lib_id "Connector:Conn_01x05_Socket")
+		(at 29.21 110.49 0)
+		(unit 1)
+		(exclude_from_sim no)
+		(in_bom yes)
+		(on_board yes)
+		(dnp no)
+		(fields_autoplaced yes)
+		(property "Reference" "J7"
+			(at 30.48 109.2199 0)
+			(effects
+				(font
+					(size 1.27 1.27)
+				)
+				(justify left)
+			)
+		)
+		(property "Value" "Conn_01x05_Socket"
+			(at 30.48 111.7599 0)
+			(effects
+				(font
+					(size 1.27 1.27)
+				)
+				(justify left)
+				(hide yes)
+			)
+		)
+		(property "Footprint" ""
+			(at 29.21 110.49 0)
+			(effects
+				(font
+					(size 1.27 1.27)
+				)
+				(hide yes)
+			)
+		)
+		(property "Datasheet" "~"
+			(at 29.21 110.49 0)
+			(effects
+				(font
+					(size 1.27 1.27)
+				)
+				(hide yes)
+			)
+		)
+		(property "Description" "Generic connector, single row, 01x05, script generated"
+			(at 29.21 110.49 0)
+			(effects
+				(font
+					(size 1.27 1.27)
+				)
+				(hide yes)
+			)
+		)
+		(pin "5"
+		)
+		(pin "3"
+		)
+		(pin "1"
+		)
+		(pin "2"
+		)
+		(pin "4"
+		)
+		(instances
+			(project "mainboard"
+				(path "/d7035e05-04e9-4d00-b42e-d5291b634456"
+					(reference "J7")
+					(unit 1)
+				)
+			)
+		)
+	)
+	(symbol
 		(lib_id "Device:R_Potentiometer")
 		(at 81.28 68.58 0)
@@
 			)
 		)
-		(property "Footprint" "Capacitor_THT:CP_Radial_D12.5mm_P5.00mm"
+		(property "Footprint" "Capacitor_THT:CP_Radial_D5.0mm_P2.00mm"
 			(at 102.5652 184.15 0)
 			(effects
@@
 			)
 		)
-		(property "Footprint" ""
+		(property "Footprint" "Eurorack:AudioJack_3.5mm"
 			(at 191.77 106.68 0)
 			(effects
@@
 			)
 		)
-		(property "Footprint" "Capacitor_THT:CP_Radial_D12.5mm_P5.00mm"
+		(property "Footprint" "Capacitor_THT:CP_Radial_D5.0mm_P2.00mm"
 			(at 102.5652 191.77 0)
 			(effects

Commit message: stuff
Parts:
- added J10, J9: Conn_01x05_Pin, symbol Connector:Conn_01x05_Pin
Other:
- moved on the sheet: C1, C2, C3, C4, J1, J2, J3, J4, J5, J6, J7, J8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
